File: esquematico.brd (EAGLE design)
At the start: 61.1 x 80.5 mm, 38 parts, among them IC1 TS321IDBVR, IC2 ESP32-S3-WROOM-1-N16R8, IC3 MAX30102EFD+T, IC4 MCP73831T-2ACI_OT, IC5 LP38692MP-3.3_NOPB, IC6 CP2102N-A02-GQFN20R, J1 UJ20-C-H-G-MSMT-P16-TR-67, J2 B2B-PH-K-S_LF__SN_, J4 PJ-202AH, M1 ELECTRET_MICROPHON-WM.64PN

Commit message: esquematico actualizado
Parts:
- removed IC6: CP2102N-A02-GQFN20R, CP2102N-A02-GQFN20R:CP2102NA02GQFN20
- removed J2: B2B-PH-K-S_LF__SN_, B2B-PH-K-S_LF__SN_:SHDR2W50P0X200_1X2_590X450X600
- removed J4: PJ-202AH, PJ-202AH:PJ202AH
- removed R13: 10K, 0805S8F1202P5E:RESC2013X65N
- removed S1, S2: MJTP1212C, MJTP1212C:MJTP1212C
- added J5: 1769, 1769:1769
- added S3: PCM13SMTR, PCM13SMTR:SW_PCM13SMTR
- added S4, S5: DTSM-61N-V-T_R, DTSM-61N-V-T_R:DTSM61NVTR
Connections:
- removed net GND3: C8.1, J2.1
- removed net N$10: J1.A12
- removed net N$12: C7.2, D2.C, IC4.4
- removed net N$15: IC6.9, R13.2
- removed net RESET32: C10.1, IC2.3, S1.1
- new net N$7: C8.1, J5.1
- net +3V3: no longer IC6.6, IC6.7, J4.1, R13.1
- net +5V: now also C7.2, D2.C, IC4.4, S3.4
- net +BATT: now also S3.2; no longer J4.2
- net DN1: no longer IC6.5
- net DP1: no longer IC6.4
- net GND: now also J1.A12, J5.2, S4.3, S5.1; no longer IC6.2, J2.2, S1.3, S2.1
- net GND1: now also S5.3; no longer S2.3
- net INT1: now also C10.1, IC2.3, S4.1
- net N$6: now also S3.3; no longer J4.3
- net RXD: no longer IC6.17
- net TXD: no longer IC6.18
