File: esquematico.sch (EAGLE design)
At the start: 38 parts, among them IC1 TS321IDBVR, IC2 ESP32-S3-WROOM-1-N16R8, IC3 MAX30102EFD+T, IC4 MCP73831T-2ACI_OT, IC5 LP38692MP-3.3_NOPB, IC6 CP2102N-A02-GQFN20R, J1 UJ20-C-H-G-MSMT-P16-TR-67, J2 B2B-PH-K-S_LF__SN_, J4 PJ-202AH, M1 ELECTRET_MICROPHON-WM.64PN

Commit message: esquematico actualizado
Parts:
- removed IC6: CP2102N-A02-GQFN20R, CP2102N-A02-GQFN20R:CP2102N-A02-GQFN20R
- removed J2: B2B-PH-K-S_LF__SN_, B2B-PH-K-S_LF__SN_:B2B-PH-K-S_LF__SN_
- removed J4: PJ-202AH, PJ-202AH:PJ-202AH
- removed R13: 10K, 0805S8F1202P5E:0805S8F1202P5E
- removed S1, S2: MJTP1212C, MJTP1212C:MJTP1212C
- added J5: 1769, 1769:1769
- added S3: PCM13SMTR, PCM13SMTR:PCM13SMTR
- added S4, S5: DTSM-61N-V-T_R, DTSM-61N-V-T_R:DTSM-61N-V-T_R
Connections:
- removed net GND3: C8.1, J2.1
- removed net N$10: J1.GND_1
- removed net N$12: C7.2, D2.C, IC4.VDD
- removed net N$15: IC6.RSTB, R13.2
- removed net RESET32: C10.1, IC2.EN, S1.COM_1
- new net N$7: C8.1, J5.1
- net +3V3: no longer IC6.VDD, IC6.VREGIN, J4.1, R13.1
- net +5V: now also C7.2, D2.C, IC4.VDD, S3.4
- net +BATT: now also S3.2; no longer J4.2
- net DN1: no longer IC6.D-
- net DP1: no longer IC6.D+
- net GND: now also J1.GND_1, J5.2, S4.NO_1, S5.COM_1; no longer IC6.GPIO.0_/_CLK, J2.2, S1.NO_1, S2.COM_1
- net GND1: now also S5.NO_1; no longer S2.NO_1
- net INT1: now also C10.1, IC2.EN, S4.COM_1
- net N$6: now also S3.3; no longer J4.3
- net RXD: no longer IC6.RXD
- net TXD: no longer IC6.TXD
Other:
- note removed: "+BATT"
- note removed: "COMUNICACION SERIAL UART"
- moved on the sheet: C11, C8, R11
