File: circuito1.1.sch (EAGLE design)
At the start: 38 parts

Commit message: Se terminó el PCB
Parts:
- removed CONECTOR-MICRO: B2B-PH-SM4-TB_LF__SN_, B2B-PH-SM4-TB_LF__SN_:B2B-PH-SM4-TB_LF__SN_
- removed SV1: (no value), con-lstb:MA03-1
- added MICRO: (no value), con-lstb:MA03-1
- renumbered AMPLIFICADOR to AMP, CONECTOR-USB-C to USB-C, PULSADOR-FLASH to FLASH, PULSADOR-RESET to RESET, REGULADOR to REGV, REGULADOR-BATERIA to C-BATT
Connections:
- net +5V renamed VDD
- removed net PIN24: ESP32-S3.IO47
- new net D1+: ESP32-S3.IO21, USB-C.D1+
- new net D1-: ESP32-S3.IO47, USB-C.D1-
- net GND: now also MICRO.2; no longer CONECTOR-MICRO.1
- net N$11: now also MICRO.3; no longer CONECTOR-MICRO.2
