File: circuito1.1.brd (EAGLE design)
At the start: 56 x 82.5 mm, 38 parts

Commit message: Se terminó el PCB
Parts:
- removed CONECTOR-MICRO: B2B-PH-SM4-TB_LF__SN_, B2B-PH-SM4-TB_LF__SN_:B2B-PH-SM4-TB
- removed CONECTOR-USB-C: CX90B-16P1, CX90B-16P1:HIROSE_CX90B-16P1
- removed REGULADOR-BATERIA: MCP73831T-2ACI_OT, MCP73831T-2ACI_OT:SOT95P270X145-5N
- removed SV1: (no value), con-lstb:MA03-1
- added C-BATT: MCP73831T-2ACI_OT, MCP73831T-2ACI_OT:SOT95P270X145-5N
- added MICRO: (no value), con-lstb:MA03-1
- added USB-C: CX90B-16P1, CX90B-16P1:HIROSE_CX90B-16P1
- moved R12 27.8 mm to (68.3, 10.1)
- moved R13 25.0 mm to (72.1, 10.2)
- moved C7 21.5 mm to (79.7, 14.5)
- moved SWITCH 20.3 mm to (92.4, 2.30)
- moved R9 17.7 mm to (79.7, 18.2)
- moved C8 14.2 mm to (53.0, 11.1)
- moved LED 10.4 mm to (58.2, 18.4), turned to 180 degrees
- moved R6 9.16 mm to (62.6, 18.3)
- moved R4 3.37 mm to (48.6, 36.0)
- moved OLED 3.18 mm to (48.4, 30.1)
- moved C4 2.67 mm to (48.5, 39.1)
- moved ESP32-S3 2.36 mm to (85.4, 65.2)
- moved R3 1.98 mm to (48.6, 42.2)
- renumbered AMPLIFICADOR to AMP, PULSADOR-FLASH to FLASH, PULSADOR-RESET to RESET, REGULADOR to REGV
Connections:
- removed net +5V: C7.2, CONECTOR-USB-C.A4, CONECTOR-USB-C.A9, CONECTOR-USB-C.B4, CONECTOR-USB-C.B9, LED.2, REGULADOR-BATERIA.4, SWITCH.4
- removed net PIN24: ESP32-S3.24
- new net D1+: ESP32-S3.23, USB-C.A6
- new net D1-: ESP32-S3.24, USB-C.A7
- new net VDD: C-BATT.4, C7.2, LED.2, SWITCH.4, USB-C.A4, USB-C.A9, USB-C.B4, USB-C.B9
- net BATT+: now also C-BATT.3; no longer REGULADOR-BATERIA.3
- net GND: now also C-BATT.2, MICRO.2, USB-C.A1, USB-C.A12, USB-C.B1, USB-C.B12; no longer CONECTOR-MICRO.1, CONECTOR-USB-C.A1, CONECTOR-USB-C.A12, CONECTOR-USB-C.B1, CONECTOR-USB-C.B12, REGULADOR-BATERIA.2
- net N$11: now also MICRO.3; no longer CONECTOR-MICRO.2
- net N$13: now also C-BATT.5; no longer REGULADOR-BATERIA.5
- net N$3: now also C-BATT.1; no longer REGULADOR-BATERIA.1
- net N$8: now also USB-C.A5; no longer CONECTOR-USB-C.A5
- net N$9: now also USB-C.B5; no longer CONECTOR-USB-C.B5
Routing:
- net D1-: track 0.00 -> 83.3 mm, vias 0 -> 2
- net PIN24: track 81.2 -> 0.00 mm, vias 2 -> 0
- net D1+: track 0.00 -> 76.8 mm, vias 0 -> 2
- net VDD: track 0.00 -> 74.2 mm, vias 0 -> 6
- net BATT+: track 0.00 -> 61.3 mm, vias 0 -> 2
- net N$5023: track 91.4 -> 69.7 mm, vias 2 -> 4
- net N$8: track 25.4 -> 5.55 mm
- net +3V3: track 232.1 -> 213.0 mm, vias 3 -> 7
- net N$9: track 22.3 -> 5.12 mm
- net N$6: track 55.5 -> 45.2 mm
- net EN: track 25.7 -> 16.4 mm
- net OUT: track 100.4 -> 91.7 mm, vias 0 -> 2
- net SDA: track 85.6 -> 77.0 mm
- net N$13: track 11.3 -> 4.15 mm
- net N$11: track 23.1 -> 16.5 mm
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Other:
- board size 56 x 82.5 mm -> 57.5 x 83.9 mm
- board text added: "C:/Users/user/OneDrive/Escritorio/LOGOTIPO1.3.bmp"
- board text added: "Valentina Restrepo Kevin Moreno David Betancur"

Commit message: fix: revision pcb
Parts:
- moved R12 0.70 mm to (67.6, 10.1)
- moved LED 0.15 mm to (58.2, 18.3)
- moved R9 0.13 mm to (79.7, 18.3)
Routing:
- net OUT: track 91.7 -> 86.5 mm
- net N$4: track 19.5 -> 21.1 mm
- net VDD: track 74.2 -> 72.9 mm
- net N$5023: track 69.7 -> 70.4 mm
- net INT: track 66.2 -> 65.6 mm

Commit message: Se corrigió lo que el profesor indicó
Parts:
- added C13: 100nF, C0805J104K1RACAUTO:CAPC2012X140N
- added C14: 10µF, C0805J104K1RACAUTO:CAPC2012X140N
- added REGP: LP38692MP-1.8_NOPB, LP38692MP-1.8_NOPB:SOT150P700X180-5N
- moved C5 3.76 mm to (86.0, 32.0)
Connections:
- removed net VLED: C6.2, PPG.10, PPG.9
- new net COMM: REGP.1, REGP.4
- new net VDD2: C13.2, C5.2, PPG.11, REGP.3
- net +3V3: now also C14.2, C6.2, PPG.10, PPG.4, PPG.9; no longer C5.2, PPG.11
- net GND: now also C13.1, C14.1, REGP.5; no longer PPG.4
Routing:
- net VDD2: track 0.00 -> 50.5 mm, vias 0 -> 2
- net +3V3: track 212.6 -> 234.7 mm
- net COMM: track 0.00 -> 11.9 mm, vias 0 -> 2
- net VLED: track 9.60 -> 0.00 mm
- net INT: track 65.6 -> 67.5 mm
Other:
- board text removed: "Valentina Restrepo Kevin Moreno David Betancur"
